File: energymeter.kicad_pcb (KiCad board)
At the start: 2 copper layers, 88.5 x 69.5 mm, 121 parts, among them J1 CT1, J10 CT10, J11 LINE, J12 Conn_02x09_Odd_Even, J13 Conn_02x09_Odd_Even, J2 CT2, J3 CT3, J4 CT4, J5 CT5, J6 CT6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

Commit message: Updates
Parts:
- added J14: NEUTRAL, TerminalBlock_Phoenix:TerminalBlock_Phoenix_MKDS-1,5-2_1x02_P5.00mm_Horizontal, F.Cu at (34.0, 77.5)
- moved J11 7.52 mm to (29.0, 22.8), turned to 0 degrees
- moved R63 7.52 mm to (35.0, 31.5), turned to 180 degrees
- moved R64 6.58 mm to (35.5, 34.8)
- moved R65 3.08 mm to (24.2, 31.5)
- moved R66 3.08 mm to (28.0, 31.5)
- moved R67 3.01 mm to (31.5, 31.5)
- moved T1 1.95 mm to (37.7, 40.4)
Connections:
- J11 pad 2: Net-(J11-Pin_2) -> Net-(J11-Pin_1)
- R63 pad 2: Net-(J11-Pin_2) -> Net-(R63-Pad2)
- R67 pad 1: Net-(R67-Pad1) -> Net-(R63-Pad2)
- T1 pad 2: Net-(R67-Pad1) -> Net-(J14-Pin_1)
Other:
- copper layers 2 -> 4

Commit message: Change connector, assign JLCPCB
Parts:
- added C21: 100uF, Capacitor_Tantalum_SMD:CP_EIA-3528-21_Kemet-B, F.Cu at (2.52, 1.68)
- added C31: 100uF, Capacitor_Tantalum_SMD:CP_EIA-3528-21_Kemet-B, F.Cu at (2.52, 6.03)
- added C32: 100nF, Capacitor_SMD:C_0603_1608Metric, F.Cu at (7.50, 0.76)
- J1, J10, J2, J3, J4, J5, J6, J7, J8, J9: footprint TerminalBlock_Phoenix:TerminalBlock_Phoenix_MKDS-1,5-2_1x02_P5.00mm_Horizontal -> Connector_JST:JST_XH_B2B-XH-A_1x02_P2.50mm_Vertical
- R1, R12, R13, R18, R19, R24, R25, R30, R31, R36, R37, R4, R42, R43, R48, R49, R54, R55, R60, R9: value R0 -> 0R
- moved J1 12.5 mm to (54.0, 23.0)
- moved J10 9.25 mm to (55.8, 77.7)
- moved J2 9.00 mm to (63.5, 23.0)
- moved J9 6.25 mm to (65.8, 77.7)
- moved J3 5.50 mm to (73.0, 23.0)
- moved J8 3.25 mm to (75.8, 77.7)
- moved J4 2.75 mm to (83.2, 23.0)
- moved J6 2.75 mm to (95.8, 77.7)
- moved J5 0.50 mm to (93.0, 23.0)
- moved J7 0.25 mm to (85.8, 77.7)

Commit message: After layout
Parts:
- removed C22: 100nF, Capacitor_SMD:C_0603_1608Metric
- removed D1: SS36, Diode_SMD:D_SMA
- removed U2: XL1509-3.3, Package_SO:SOIC-8_3.9x4.9mm_P1.27mm
- moved C21 136.0 mm to (91.0, 105.0)
- moved C31 129.1 mm to (91.0, 100.0)
- moved C32 116.9 mm to (82.4, 90.5), turned to 180 degrees
- moved J11 88.4 mm to (41.5, 110.3)
- moved R65 72.4 mm to (36.1, 102.9), turned to -90 degrees
- moved R66 68.0 mm to (36.1, 99.0), turned to -90 degrees
- moved R64 64.9 mm to (40.7, 99.5)
- moved J6 64.3 mm to (41.0, 44.0), turned to 0 degrees
- moved R63 63.8 mm to (40.7, 95.0), turned to 90 degrees
- moved R67 63.7 mm to (36.1, 95.0), turned to -90 degrees
- moved U3 61.3 mm to (82.3, 101.2)
- moved R33 60.3 mm to (40.7, 51.2), turned to 0 degrees
- moved T1 60.1 mm to (45.5, 100.1), turned to 90 degrees
- moved R35 59.2 mm to (40.0, 53.9), turned to -90 degrees
- moved C12 57.0 mm to (40.8, 56.7), turned to 0 degrees
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Connections:
- U1 pad 45: unconnected-(U1-IN4-Pad45) -> /IN4
- U1 pad 47: /IP5 -> /IN5
Routing:
- net +5V: track 0.00 -> 149.5 mm, vias 0 -> 1
- net GND: track 0.00 -> 117.0 mm, vias 0 -> 27
- net /SDI: track 0.00 -> 113.6 mm, vias 0 -> 3
- net /SDO: track 0.00 -> 86.1 mm, vias 0 -> 2
- net /SCLK: track 0.00 -> 82.6 mm, vias 0 -> 2
- net +3.3V: track 0.00 -> 79.1 mm
- net /IP6: track 0.00 -> 70.4 mm, vias 0 -> 2
- net /IN6: track 0.00 -> 67.9 mm, vias 0 -> 2
- net /CS6: track 0.00 -> 67.3 mm
- net /CS5: track 0.00 -> 66.3 mm
- net /IN7: track 0.00 -> 66.2 mm, vias 0 -> 2
- net /CS4: track 0.00 -> 65.5 mm
- net /CS3: track 0.00 -> 64.0 mm
- net /CS2: track 0.00 -> 62.9 mm
- net /IP1: track 0.00 -> 62.2 mm, vias 0 -> 2
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- added copper zone on In1.Cu, net GND
Other:
- board size 88.5 x 69.5 mm -> 67 x 86 mm
- board text added: "3Mod Width 53.0mm Height 90.0mm"
- board text added: "4Mod Width 71.0 Height 90.0"

Commit message: Board cleanup
Routing:
- net GND: track 117.0 -> 105.9 mm
- net /IN3: track 56.5 -> 47.7 mm
- net /IN2: track 61.1 -> 54.0 mm
- net /IP1: track 62.2 -> 55.3 mm
- net +3.3V: track 79.1 -> 80.3 mm
- net Net-(R63-Pad2): track 5.46 -> 4.61 mm
- net /IRQ1: track 55.3 -> 54.5 mm

Commit message: First order
Parts:
- J12, J13: value Conn_02x09_Odd_Even -> Conn_02x10_Odd_Even; footprint Connector_PinHeader_2.54mm:PinHeader_2x09_P2.54mm_Vertical -> Connector_PinHeader_2.54mm:PinHeader_2x10_P2.54mm_Vertical
Routing:
- net GND: track 105.9 -> 108.6 mm
- net /IP6: track 70.3 -> 69.6 mm
- net /IP10: track 42.1 -> 41.4 mm
